Commit message: [ouster-imu.urdf.xacro] Add namespace

File: urdf/ouster-imu.urdf.xacro (robot description, xacro)
@@ -1,3 +1,6 @@
-<robot name="danieli-drone">
+<?xml version="1.0"?>
+<robot name="danieli-drone" xmlns:xacro="http://ros.org/wiki/xacro">
+  <xacro:arg name="namespace" default="none"/>
+  <xacro:property name="namespace" value="$(arg namespace)" />
   <material name="orange">
     <color rgba="1.0 0.5 0.2 1" />
@@ -6,5 +9,5 @@
     <color rgba="0.2 0.2 0.2 1" />
   </material>
-  <link name="danieli2/imu_link">
+  <link name="${namespace}/imu_link">
     <visual>
       <origin xyz="0.0 0.0 0.0" />
@@ -33,16 +36,16 @@
     </visual>
   </link>
-  <link name="base_link" />
-  <joint name="imu_link_joint" type="fixed">
-    <parent link="base_link" />
-    <child link="danieli2/imu_link" />
+  <link name="${namespace}/base_link" />
+  <joint name="${namespace}/imu_link_joint" type="fixed">
+    <parent link="${namespace}/base_link" />
+    <child link="${namespace}/imu_link" />
     <origin xyz="0 0 0" rpy="0 0 0" />
   </joint>
-  <joint name="ouster_link_joint" type="fixed">
-    <parent link="base_link" />
+  <joint name="${namespace}/ouster_link_joint" type="fixed">
+    <parent link="${namespace}/base_link" />
     <child link="os_lidar" />
     <origin xyz="0.08 0. -0.1578" rpy="3.151592653589793 0.3023284641020683 0." />
   </joint>
-  <joint name="os_imu_link_joint" type="fixed">
+  <joint name="${namespace}/os_imu_link_joint" type="fixed">
     <parent link="os_lidar" />
     <child link="os_imu" />
